File: kicad/can.kicad_sch (KiCad schematic)
At the start: 11 parts, among them U7 TCAN334

Commit message: removed load terminal & circuit
Parts:
- R11: footprint LibreSolar:R_1206_3216 -> Resistor_SMD:R_1206_3216Metric
Changed lines of the file:
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@@
       (effects (font (size 1.27 1.27)) (justify left))
     )
-    (property "Footprint" "LibreSolar:R_1206_3216" (id 2) (at 114.935 99.06 0)
+    (property "Footprint" "Resistor_SMD:R_1206_3216Metric" (id 2) (at 114.935 99.06 0)
       (effects (font (size 1.27 1.27)) hide)
     )

Commit message: pcb minor fixes, updated bom files, updated project name
Other:
- title: MPPT 2420 HC -> MPPT 4820 HC
Changed lines of the file:
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@@
   (paper "A4")
   (title_block
-    (title "MPPT 2420 HC")
+    (title "MPPT 4820 HC")
     (date "2021-01-06")
     (rev "0.2.3")
