File: kicad/mcu.kicad_sch (KiCad schematic)
At the start: 37 parts, among them J7 UEXT, P1 CONN_01X02, U2 STM32G431CBTx, U6 W25Q80DVS, Y1 8MHz

Commit message: pcb minor fixes, updated bom files, updated project name
Other:
- title: MPPT 2420 HC -> MPPT 4820 HC
Changed lines of the file:
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@@
   (paper "A4")
   (title_block
-    (title "MPPT 2420 HC")
+    (title "MPPT 4820 HC")
     (date "2021-03-17")
     (rev "0.2.3")
