File: kicad/mppt-4820-hc.kicad_sch (KiCad schematic)
At the start: 16 parts, among them J1 MKDS 5/ 2-9,5, J2 MKDS 5/ 2-9,5, J4 8P8C, J5 8P8C

Commit message: pcb minor fixes, updated bom files, updated project name
Other:
- title: MPPT 2420 HC -> MPPT 4820 HC
Changed lines of the file:
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@@
   (paper "A4")
   (title_block
-    (title "MPPT 2420 HC")
+    (title "MPPT 4820 HC")
     (date "2021-01-06")
     (rev "0.2.3")

Commit message: some DRC check errors fixes (prototype 1)
Parts:
- F1: footprint LibreSolar:NULL -> LibreSolar:Eaton_S-4000
Changed lines of the file:
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@@
       (effects (font (size 1.27 1.27)))
     )
-    (property "Footprint" "LibreSolar:NULL" (at 198.12 45.72 0)
+    (property "Footprint" "LibreSolar:Eaton_S-4000" (at 198.12 45.72 0)
       (effects (font (size 1.27 1.27)) hide)
     )
